File: interface_board/interface_board.kicad_sch (KiCad schematic)
At the start: 0 parts

Commit message: Add interface board PCB design
Parts:
- added D_ACT: GREEN, LED_SMD:LED_0805_2012Metric_Pad1.15x1.40mm_HandSolder, symbol Device:LED_Filled
- added D_PWR: RED, LED_SMD:LED_0805_2012Metric_Pad1.15x1.40mm_HandSolder, symbol Device:LED_Filled
- added J1: FPGA_devboard, Connector_PinSocket_2.54mm:PinSocket_2x22_P2.54mm_Vertical, symbol Connector_Generic:Conn_02x22_Odd_Even
- added J2: 5V_PWR, Connector_PinHeader_2.54mm:PinHeader_1x02_P2.54mm_Vertical, symbol Connector_Generic:Conn_01x02
- added R22, R23: 680, Resistor_SMD:R_0805_2012Metric_Pad1.20x1.40mm_HandSolder, symbol Device:R
Connections:
- new net: D_ACT.2 (A), R23.2
- new net: D_PWR.2 (A), R22.2
- new net +3V3: J1.1 (Pin_1), J1.2 (Pin_2)
- new net +5V: J2.1 (Pin_1)
- new net ACTION: J1.6 (Pin_6), R23.1
- new net ATN_IN: J1.8 (Pin_8)
- new net CLK_IN: J1.10 (Pin_10)
- new net CLK_OUT: J1.16 (Pin_16)
- new net DATA_IN: J1.11 (Pin_11)
- new net DATA_OUT: J1.15 (Pin_15)
- new net DIR: J1.32 (Pin_32)
- new net DRVSA: J1.36 (Pin_36)
- new net DRVSB: J1.35 (Pin_35)
- new net DSKCHG: J1.23 (Pin_23)
- new net GND: D_ACT.1 (K), D_PWR.1 (K), J1.13 (Pin_13), J1.14 (Pin_14), J1.21 (Pin_21), J1.22 (Pin_22), J1.29 (Pin_29), J1.30 (Pin_30), J1.37 (Pin_37), J1.38 (Pin_38), J2.2 (Pin_2)
- new net INDEX: J1.28 (Pin_28)
- new net MOTEA: J1.40 (Pin_40)
- new net MOTEB: J1.33 (Pin_33)
- new net PWR: J1.5 (Pin_5), R22.1
- new net RDATA: J1.24 (Pin_24)
- new net REDWC_IN: J1.27 (Pin_27)
- new net REDWC_OUT: J1.39 (Pin_39)
- new net RESET_IN: J1.9 (Pin_9)
- new net SIDE1: J1.20 (Pin_20)
- new net SQR_IN: J1.7 (Pin_7)
- new net SRQ_OUT: J1.17 (Pin_17)
- new net STEP: J1.31 (Pin_31)
- new net TRK00: J1.26 (Pin_26)
- new net WDATE: J1.18 (Pin_18)
- new net WGATE: J1.19 (Pin_19)
- new net WPT: J1.25 (Pin_25)
- no-connect marks 0 -> 8
Other:
- added sheet IBM PC floppy interface (floppy.kicad_sch)
- added sheet Serial interface (serial.kicad_sch)

Commit message: Finish interface board PCB
Parts:
- J2: footprint Connector_PinHeader_2.54mm:PinHeader_1x02_P2.54mm_Vertical -> Connector_PinHeader_2.54mm:PinHeader_1x09_P2.54mm_Vertical; symbol Connector_Generic:Conn_01x02 -> Connector_Generic:Conn_01x09
- renumbered D_ACT to D_ACT1, D_PWR to D_PWR1
Connections:
- net +5V: now also J2.2 (Pin_2); no longer J2.1 (Pin_1)
- net ACTION: now also J1.5 (Pin_5); no longer J1.6 (Pin_6)
- net ATN_IN: now also J1.7 (Pin_7); no longer J1.8 (Pin_8)
- net CLK_IN: now also J1.9 (Pin_9); no longer J1.10 (Pin_10)
- net CLK_OUT: now also J1.15 (Pin_15); no longer J1.16 (Pin_16)
- net DATA_IN: now also J1.12 (Pin_12); no longer J1.11 (Pin_11)
- net DATA_OUT: now also J1.16 (Pin_16); no longer J1.15 (Pin_15)
- net DIR: now also J1.39 (Pin_39); no longer J1.32 (Pin_32)
- net DRVSA: now also J1.41 (Pin_41); no longer J1.36 (Pin_36)
- net DRVSB: now also J1.42 (Pin_42); no longer J1.35 (Pin_35)
- net DSKCHG: now also J1.24 (Pin_24); no longer J1.23 (Pin_23)
- net GND: now also J2.1 (Pin_1); no longer J2.2 (Pin_2)
- net INDEX: now also J1.27 (Pin_27); no longer J1.28 (Pin_28)
- net MOTEA: now also J1.43 (Pin_43); no longer J1.40 (Pin_40)
- net MOTEB: now also J1.40 (Pin_40); no longer J1.33 (Pin_33)
- net PWR: now also J1.6 (Pin_6); no longer J1.5 (Pin_5)
- net RDATA: now also J1.23 (Pin_23); no longer J1.24 (Pin_24)
- net REDWC_IN: now also J1.28 (Pin_28); no longer J1.27 (Pin_27)
- net REDWC_OUT: now also J1.44 (Pin_44); no longer J1.39 (Pin_39)
- net RESET_IN: now also J1.10 (Pin_10); no longer J1.9 (Pin_9)
- net SIDE1: now also J1.19 (Pin_19); no longer J1.20 (Pin_20)
- net SQR_IN: now also J1.8 (Pin_8); no longer J1.7 (Pin_7)
- net SRQ_OUT: now also J1.18 (Pin_18); no longer J1.17 (Pin_17)
- net STEP: now also J1.32 (Pin_32); no longer J1.31 (Pin_31)
- net TRK00: now also J1.25 (Pin_25); no longer J1.26 (Pin_26)
- net WDATE: now also J1.17 (Pin_17); no longer J1.18 (Pin_18)
- net WGATE: now also J1.20 (Pin_20); no longer J1.19 (Pin_19)
- net WPT: now also J1.26 (Pin_26); no longer J1.25 (Pin_25)
- no-connect marks 8 -> 15
