File: interface_board/floppy.kicad_sch (KiCad schematic)
At the start: 24 parts, among them J4 IBM PC floppy disk drive conn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, Q1 BC337, U1 74LS06, U2 74LVC14, U3 74LS06, U4 74LVC14

Commit message: Finish interface board PCB
Parts:
- J4: footprint Connector_PinHeader_2.54mm:PinHeader_2x17_P2.54mm_Vertical -> Connector_IDC:IDC-Header_2x17_P2.54mm_Vertical
- Q1: footprint Package_TO_SOT_THT:TO-92_Inline -> Package_TO_SOT_THT:TO-92_Inline_Wide
Changed lines of the file:
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@@
       (effects (font (size 1.27 1.27)) (justify left))
     )
-    (property "Footprint" "Package_TO_SOT_THT:TO-92_Inline" (id 2) (at 205.74 61.595 0)
+    (property "Footprint" "Package_TO_SOT_THT:TO-92_Inline_Wide" (id 2) (at 205.74 61.595 0)
       (effects (font (size 1.27 1.27) italic) (justify left) hide)
     )
@@
     (property "Reference" "J4" (id 0) (at 245.11 35.56 0))
     (property "Value" "IBM PC floppy disk drive connector" (id 1) (at 245.11 38.1 0))
-    (property "Footprint" "Connector_PinHeader_2.54mm:PinHeader_2x17_P2.54mm_Vertical" (id 2) (at 246.38 62.23 0)
-      (effects (font (size 1.27 1.27)) hide)
-    )
+    (property "Footprint" "Connector_IDC:IDC-Header_2x17_P2.54mm_Vertical" (id 2) (at 246.38 62.23 0)
+      (effects (font (size 1.27 1.27)) hide)
+    )

Commit message: Add schematics for appendix, add sketch to diploma, simulate startup in isim
Other:
- company: (none) -> Weisz Pál
- title: (none) -> FPGA - C64 Floppy drive interface board
Changed lines of the file:
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@@
 (kicad_sch (version 20211123) (generator eeschema)
   (paper "A4")
+  (title_block
+    (title "FPGA - C64 Floppy drive interface board")
+    (date "2022-09-14")
+    (rev "1")
+    (company "Weisz Pál")
+  )
   (junction (at 137.16 87.63) (diameter 0) (color 0 0 0 0)
   )
