File: interface_board/serial.kicad_sch (KiCad schematic)
At the start: 10 parts, among them J3 Serial IEEE-488 Bus, U1 74LS06, U2 74LVC14

Commit message: Add schematics for appendix, add sketch to diploma, simulate startup in isim
Other:
- company: (none) -> Weisz Pál
- title: (none) -> FPGA - C64 Floppy drive interface board
Changed lines of the file:
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@@
 (kicad_sch (version 20211123) (generator eeschema)
   (paper "A4")
+  (title_block
+    (title "FPGA - C64 Floppy drive interface board")
+    (date "2022-09-14")
+    (rev "1")
+    (company "Weisz Pál")
+  )
   (junction (at 166.37 135.89) (diameter 0) (color 0 0 0 0)
   )
